File: oc01.kicad_sch (KiCad schematic)
At the start: 0 parts

Commit message: Create schematic.
Parts:
- added D1: 1N5819, Diode_THT:D_DO-41_SOD81_P10.16mm_Horizontal, symbol Diode:1N5819
- added D2, D3, D4, D5: YELLOW, symbol Device:LED
- added J1, J2: ~, symbol Connector:Screw_Terminal_01x05
- added R1, R2, R3, R4: 1k, symbol Device:R
- added U1: PC847, Package_DIP:DIP-16_W7.62mm, symbol Isolator:PC847
Connections:
- new net: D4.2 (A), U1.6
- new net: D4.1 (K), R3.1
- new net: D2.1 (K), R1.1
- new net: D2.2 (A), U1.2
- new net: D5.1 (K), R4.1
- new net: D5.2 (A), U1.8
- new net: D3.1 (K), R2.1
- new net: D3.2 (A), U1.4
- new net GNDA: J2.1 (Pin_1), U1.11, U1.13, U1.15, U1.9
- new net IN1: J1.2 (Pin_2), R1.2
- new net IN2: J1.3 (Pin_3), R2.2
- new net IN3: J1.4 (Pin_4), R3.2
- new net IN4: J1.5 (Pin_5), R4.2
- new net OUT1: J2.2 (Pin_2), U1.16
- new net OUT2: J2.3 (Pin_3), U1.14
- new net OUT3: J2.4 (Pin_4), U1.12
- new net OUT4: J2.5 (Pin_5), U1.10
- new net VCC: D1.2 (A), J1.1 (Pin_1)
- new net VCCIN: D1.1 (K), U1.1, U1.3, U1.5, U1.7
Other:
- note added: "Allowed VCC: 5-24 V (1-20 mA optocoupler current)"
- note added: "D1+U1+LED forward voltage = ~3.85 V"
- company: (none) -> Model Railroader Club Brno I – KMŽ Brno I – https://kmz-brno.cz/
- title: (none) -> OC01 - Universal optocoupler module

Commit message: Add footprints.
Parts:
- D1: footprint Diode_THT:D_DO-41_SOD81_P10.16mm_Horizontal -> Diode_SMD:D_SOD-123
- D2, D3, D4, D5: footprint (none) -> LED_SMD:LED_0805_2012Metric_Pad1.15x1.40mm_HandSolder
- J1, J2: footprint (none) -> TerminalBlock_4Ucon:TerminalBlock_4Ucon_1x05_P3.50mm_Horizontal
- R1, R2, R3, R4: footprint (none) -> Resistor_SMD:R_0805_2012Metric_Pad1.20x1.40mm_HandSolder
- U1: footprint Package_DIP:DIP-16_W7.62mm -> Package_DIP:DIP-16_W7.62mm_LongPads
Changed lines of the file:
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@@
 			)
 		)
-		(property "Footprint" "Package_DIP:DIP-16_W7.62mm"
+		(property "Footprint" "Package_DIP:DIP-16_W7.62mm_LongPads"
 			(at 105.41 72.39 0)
 			(effects
@@
 			)
 		)
-		(property "Footprint" ""
+		(property "Footprint" "Resistor_SMD:R_0805_2012Metric_Pad1.20x1.40mm_HandSolder"
 			(at 68.58 68.072 90)
 			(effects
@@
 			)
 		)
-		(property "Footprint" ""
+		(property "Footprint" "Resistor_SMD:R_0805_2012Metric_Pad1.20x1.40mm_HandSolder"
 			(at 68.58 37.592 90)
 			(effects
@@
 			)
 		)
-		(property "Footprint" "Package_DIP:DIP-16_W7.62mm"
+		(property "Footprint" "Package_DIP:DIP-16_W7.62mm_LongPads"
 			(at 105.41 41.91 0)
 			(effects
@@
 			)
 		)
-		(property "Footprint" "Diode_THT:D_DO-41_SOD81_P10.16mm_Horizontal"
+		(property "Footprint" "Diode_SMD:D_SOD-123"
 			(at 77.47 38.735 0)
 			(effects
@@
 			)
 		)
-		(property "Footprint" ""
+		(property "Footprint" "LED_SMD:LED_0805_2012Metric_Pad1.15x1.40mm_HandSolder"
 			(at 86.36 39.37 0)
 			(effects
@@
 			)
 		)
-		(property "Footprint" ""
+		(property "Footprint" "LED_SMD:LED_0805_2012Metric_Pad1.15x1.40mm_HandSolder"
 			(at 86.36 85.09 0)
 			(effects
@@
 			)
 		)
-		(property "Footprint" ""
+		(property "Footprint" "LED_SMD:LED_0805_2012Metric_Pad1.15x1.40mm_HandSolder"
 			(at 86.36 69.85 0)
 			(effects
@@
 			)
 		)
-		(property "Footprint" ""
+		(property "Footprint" "Resistor_SMD:R_0805_2012Metric_Pad1.20x1.40mm_HandSolder"
 			(at 68.58 83.312 90)
 			(effects
@@
 			)
 		)
-		(property "Footprint" "Package_DIP:DIP-16_W7.62mm"
+		(property "Footprint" "Package_DIP:DIP-16_W7.62mm_LongPads"
 			(at 105.41 87.63 0)
 			(effects
@@
 			)
 		)
-		(property "Footprint" ""
+		(property "Footprint" "TerminalBlock_4Ucon:TerminalBlock_4Ucon_1x05_P3.50mm_Horizontal"
 			(at 163.83 62.23 0)
 			(effects
@@
 			)
 		)
-		(property "Footprint" ""
+		(property "Footprint" "LED_SMD:LED_0805_2012Metric_Pad1.15x1.40mm_HandSolder"
 			(at 86.36 54.61 0)
 			(effects
@@
 			)
 		)
-		(property "Footprint" ""
+		(property "Footprint" "Resistor_SMD:R_0805_2012Metric_Pad1.20x1.40mm_HandSolder"
 			(at 68.58 52.832 90)
 			(effects
@@
 			)
 		)
-		(property "Footprint" "Package_DIP:DIP-16_W7.62mm"
+		(property "Footprint" "Package_DIP:DIP-16_W7.62mm_LongPads"
 			(at 105.41 57.15 0)
 			(effects
@@
 			)
 		)
-		(property "Footprint" ""
+		(property "Footprint" "TerminalBlock_4Ucon:TerminalBlock_4Ucon_1x05_P3.50mm_Horizontal"
 			(at 35.56 62.23 0)
 			(effects

Commit message: Add mounting holes.
Parts:
- added H1, H2, H3, H4: M3, MountingHole:MountingHole_3.2mm_M3_Pad_Via, symbol Mechanical:MountingHole

Commit message: Wire PCB.
Connections:
- net GNDA: now also J2.5 (Pin_5); no longer J2.1 (Pin_1)
- net OUT1: now also J2.4 (Pin_4); no longer J2.2 (Pin_2)
- net OUT3: now also J2.2 (Pin_2); no longer J2.4 (Pin_4)
- net OUT4: now also J2.1 (Pin_1); no longer J2.5 (Pin_5)
Other:
- title: OC01 - Universal optocoupler module -> OC-01 - Universal optocoupler module
Changed lines of the file:
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@@
 	(paper "A5")
 	(title_block
-		(title "OC01 - Universal optocoupler module")
+		(title "OC-01 - Universal optocoupler module")
 		(date "2026-07-01")
 		(rev "1.0")
@@
 		(lib_id "Connector:Screw_Terminal_01x05")
 		(at 163.83 62.23 0)
+		(mirror x)
 		(unit 1)
 		(exclude_from_sim no)
@@
 		(on_board yes)
 		(dnp no)
-		(fields_autoplaced yes)
 		(property "Reference" "J2"
-			(at 165.862 61.7608 0)
+			(at 165.862 62.6992 0)
 			(effects
 				(font
@@
 		)
 		(property "Value" "~"
-			(at 165.862 63.4422 0)
-			(effects
-				(font
+			(at 165.862 61.0178 0)
+			(effects
+				(font
