File: oc40.kicad_pcb (KiCad board)
At the start: 2 copper layers, 40 x 45 mm, 16 parts, among them U1 PC847

Commit message: OC-01 -> OC-40 (4 optocouplers).
Other:
- board text added: "Universal Optocoupler OC-40"
- board text removed: "Universal Optocoupler OC-01"
Changed lines of the file:
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@@
 		(layer "Edge.Cuts")
 	)
-	(gr_text "Universal Optocoupler\nOC-01"
+	(gr_text "Universal Optocoupler\nOC-40"
 		(at 170.942 97.536 90)
 		(layer "F.SilkS")
