File: oc40.kicad_sch (KiCad schematic)
At the start: 16 parts, among them U1 PC847

Commit message: OC-01 -> OC-40 (4 optocouplers).
Other:
- title: OC-01 - Universal optocoupler module -> OC-40 - Universal optocoupler module
Changed lines of the file:
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@@
 	(paper "A5")
 	(title_block
-		(title "OC-01 - Universal optocoupler module")
-		(date "2026-07-01")
+		(title "OC-40 - Universal optocoupler module")
+		(date "2026-07-02")
 		(rev "1.0")
 		(company "Model Railroader Club Brno I – KMŽ Brno I – https://kmz-brno.cz/")
